Commit message: ros sdk 작성 완료

File: rby1/urdf/rby1_full_ros.urdf.xacro (robot description, xacro)
@@ -249,3 +249,117 @@
     <child link="left_arm_camera_color_optical_frame"/>
   </joint>
+  <!-- ================================================================
+       5. ROS2 Control
+          robot_ip is passed from bringup.launch.py via xacro mappings.
+          When robot_ip is empty (e.g. description.launch.py), the
+          ros2_control block is present but inactive — robot_state_publisher
+          ignores unknown tags.
+       ================================================================ -->
+  <ros2_control name="rby1_hardware" type="system">
+    <hardware>
+      <plugin>rby1/RBY1HardwareInterface</plugin>
+      <param name="robot_ip">$(arg robot_ip)</param>
+    </hardware>
+    <!-- Wheels: state only — mobile base is commanded via cmd_vel → SE2VelocityCommand gRPC -->
+    <joint name="right_wheel">
+      <state_interface name="position"><param name="initial_value">0.0</param></state_interface>
+      <state_interface name="velocity"/>
+    </joint>
+    <joint name="left_wheel">
+      <state_interface name="position"><param name="initial_value">0.0</param></state_interface>
+      <state_interface name="velocity"/>
+    </joint>
+    <!-- Torso: position command + state -->
+    <joint name="torso_0">
+      <command_interface name="position"/>
+      <state_interface name="position"><param name="initial_value">0.0</param></state_interface>
+    </joint>
+    <joint name="torso_1">
+      <command_interface name="position"/>
+      <state_interface name="position"><param name="initial_value">0.0</param></state_interface>
+    </joint>
+    <joint name="torso_2">
+      <command_interface name="position"/>
+      <state_interface name="position"><param name="initial_value">0.0</param></state_interface>
+    </joint>
+    <joint name="torso_3">
+      <command_interface name="position"/>
+      <state_interface name="position"><param name="initial_value">0.0</param></state_interface>
+    </joint>
+    <joint name="torso_4">
+      <command_interface name="position"/>
+      <state_interface name="position"><param name="initial_value">0.0</param></state_interface>
+    </joint>
+    <joint name="torso_5">
+      <command_interface name="position"/>
+      <state_interface name="position"><param name="initial_value">0.0</param></state_interface>
+    </joint>
+    <!-- Right arm: position command + state -->
+    <joint name="right_arm_0">
+      <command_interface name="position"/>
+      <state_interface name="position"><param name="initial_value">0.0</param></state_interface>
+    </joint>
+    <joint name="right_arm_1">
+      <command_interface name="position"/>
+      <state_interface name="position"><param name="initial_value">0.0</param></state_interface>
+    </joint>
+    <joint name="right_arm_2">
+      <command_interface name="position"/>
+      <state_interface name="position"><param name="initial_value">0.0</param></state_interface>
+    </joint>
+    <joint name="right_arm_3">
+      <command_interface name="position"/>
+      <state_interface name="position"><param name="initial_value">0.0</param></state_interface>
+    </joint>
+    <joint name="right_arm_4">
+      <command_interface name="position"/>
+      <state_interface name="position"><param name="initial_value">0.0</param></state_interface>
+    </joint>
+    <joint name="right_arm_5">
+      <command_interface name="position"/>
+      <state_interface name="position"><param name="initial_value">0.0</param></state_interface>
+    </joint>
+    <joint name="right_arm_6">
+      <command_interface name="position"/>
+      <state_interface name="position"><param name="initial_value">0.0</param></state_interface>
+    </joint>
+    <!-- Left arm: position command + state -->
+    <joint name="left_arm_0">
+      <command_interface name="position"/>
+      <state_interface name="position"><param name="initial_value">0.0</param></state_interface>
+    </joint>
+    <joint name="left_arm_1">
+      <command_interface name="position"/>
+      <state_interface name="position"><param name="initial_value">0.0</param></state_interface>
+    </joint>
+    <joint name="left_arm_2">
+      <command_interface name="position"/>
+      <state_interface name="position"><param name="initial_value">0.0</param></state_interface>
+    </joint>
+    <joint name="left_arm_3">
+      <command_interface name="position"/>
+      <state_interface name="position"><param name="initial_value">0.0</param></state_interface>
+    </joint>
+    <joint name="left_arm_4">
+      <command_interface name="position"/>
+      <state_interface name="position"><param name="initial_value">0.0</param></state_interface>
+    </joint>
+    <joint name="left_arm_5">
+      <command_interface name="position"/>
+      <state_interface name="position"><param name="initial_value">0.0</param></state_interface>
+    </joint>
+    <joint name="left_arm_6">
+      <command_interface name="position"/>
+      <state_interface name="position"><param name="initial_value">0.0</param></state_interface>
+    </joint>
+    <!-- Head: position command + state -->
+    <joint name="head_0">
+      <command_interface name="position"/>
+      <state_interface name="position"><param name="initial_value">0.0</param></state_interface>
+    </joint>
+    <joint name="head_1">
+      <command_interface name="position"/>
+      <state_interface name="position"><param name="initial_value">0.0</param></state_interface>
+    </joint>
+  </ros2_control>
 </robot>

Commit message: MoveIt 추가

File: rby1/urdf/rby1_full_ros.urdf.xacro (robot description, xacro)
@@ -19,4 +19,7 @@
   <xacro:arg name="initial_positions_file" default="initial_positions.yaml"/>
   <xacro:arg name="robot_ip"               default=""/>
+  <!-- end_effector: "inspire" (RH56E2 dexterous hand) or "original" (2-finger fixed gripper) -->
+  <xacro:arg name="end_effector"           default="inspire"/>
+  <xacro:property name="end_effector" value="$(arg end_effector)"/>
   <xacro:property name="M_PI" value="3.1415926535897931"/>
   <!-- ================================================================
@@ -27,9 +30,14 @@
   <xacro:include filename="$(find rby1)/urdf/rby1_base.urdf"/>
   <!-- ================================================================
-       2. Inspire Hand RH56E2 (Official — both hands)
-          Left:  FT_sensor_L → base_link       (urdf_left_with_force_sensor)
-          Right: FT_sensor_R → right_base_link  (urdf_right_with_force_sensor)
-       ================================================================ -->
-  <xacro:include filename="$(find rby1)/urdf/inspire_hand_ros.urdf.xacro"/>
+       2. End-Effector selection
+          inspire  : Inspire Robotics RH56E2 dexterous hands
+          original : 2-finger fixed gripper (ee_right / ee_left)
+       ================================================================ -->
+  <xacro:if value="${end_effector == 'inspire'}">
+    <xacro:include filename="$(find rby1)/urdf/inspire_hand_ros.urdf.xacro"/>
+  </xacro:if>
+  <xacro:if value="${end_effector == 'original'}">
+    <xacro:include filename="$(find rby1)/urdf/original_ee_ros.urdf.xacro"/>
+  </xacro:if>
   <!-- ================================================================
        3. ZED Camera on Head
